File: sigzil-rev1.0/sigzil-rev1.0.kicad_sch (KiCad schematic)
At the start: 81 parts, among them SW1 Keyswitch, SW10 Keyswitch, SW11 Keyswitch, SW12 Keyswitch, SW13 Keyswitch, SW14 Keyswitch, SW15 Keyswitch, SW16 Keyswitch, SW17 Keyswitch, SW18 Keyswitch, SW19 Keyswitch, SW2 Keyswitch, SW20 Keyswitch, SW21 Keyswitch, SW22 Keyswitch, SW23 Keyswitch, SW24 Keyswitch, SW25 Keyswitch, SW26 Keyswitch, SW27 Keyswitch, SW28 Keyswitch, SW29 Keyswitch, SW3 Keyswitch, SW30 Keyswitch, SW31 Keyswitch, SW32 Keyswitch, SW33 Keyswitch, SW34 Keyswitch, SW35 Keyswitch, SW4 Keyswitch, SW5 Keyswitch, SW6 Keyswitch, SW7 Keyswitch, SW8 Keyswitch, SW9 Keyswitch, U1 Arduino_Pro_Micro

Commit message: WIP WIP
Parts:
- SW1, SW15, SW22, SW33, SW8: footprint Sigzil:MX_PCB_1.25u -> Sigzil:MXOnly_Led_1.25u
- SW10, SW11, SW12, SW13, SW16, SW17, SW18, SW19, SW2, SW20, SW21, SW23, SW24, SW25, SW26, SW27, SW28, SW29, SW3, SW30, SW31, SW32, SW4, SW5, SW6, SW7, SW9: footprint Sigzil:MX_PCB_1.00u -> Sigzil:MXOnly_Led_1.00u
- SW14: footprint Sigzil:MX_PCB_1.25u -> Sigzil:MXOnly_Led_1.25u_90deg
- SW34, SW35: footprint Sigzil:MX_PCB_1.25u_90deg -> Sigzil:MXOnly_Led_1.25u_90deg
Connections:
- net GND: now also SW35.4
- net BACKLIGHT: now reaches U1.7 (4/PD4)
- net BACKLIGHT: now also SW1.3
- new net: SW5.4, SW6.3
- new net: SW6.4, SW7.3
- new net: SW31.4, SW32.3
- new net: SW32.4, SW33.3
- new net: SW11.3, SW12.4
- new net: SW10.3, SW11.4
- new net: SW15.4, SW16.3
- new net: SW16.4, SW17.3
- new net: SW34.4, SW35.3
- new net: SW24.3, SW25.4
- new net: SW23.3, SW24.4
- new net: SW12.3, SW13.4
- new net: SW25.3, SW26.4
- new net: SW14.3, SW7.4
- new net: SW13.3, SW14.4
- new net: SW17.4, SW18.3
- new net: SW18.4, SW19.3
- new net: SW33.4, SW34.3
- new net: SW1.4, SW2.3
- new net: SW2.4, SW3.3
- new net: SW21.4, SW28.3
- new net: SW27.3, SW28.4
- new net: SW19.4, SW20.3
- new net: SW20.4, SW21.3
- new net: SW3.4, SW4.3
- new net: SW30.4, SW31.3
- new net: SW22.4, SW29.3
- new net: SW29.4, SW30.3
- new net: SW22.3, SW23.4
- new net: SW8.3, SW9.4
- new net: SW15.3, SW8.4
- new net: SW26.3, SW27.4
- new net: SW4.4, SW5.3
- new net: SW10.4, SW9.3
- no-connect marks 5 -> 4
